Commit message: add `xmlns:xacro`

File: urdf/sinsei_umiusi_control/can.urdf.xacro (robot description, xacro)
@@ -1,4 +1,4 @@
 <?xml version="1.0" encoding="UTF-8"?>
-<xacro:macro name="can" params="with_thruster">
+<xacro:macro xmlns:xacro="http://www.ros.org/wiki/xacro" name="can" params="with_thruster">
   <ros2_control name="can" type="system">
     <hardware>

File: urdf/sinsei_umiusi_control/headlights.urdf.xacro (robot description, xacro)
@@ -1,4 +1,4 @@
 <?xml version="1.0" encoding="UTF-8"?>
-<xacro:macro name="headlights">
+<xacro:macro xmlns:xacro="http://www.ros.org/wiki/xacro" name="headlights">
   <ros2_control name="headlights" type="actuator">
     <hardware>

File: urdf/sinsei_umiusi_control/imu.urdf.xacro (robot description, xacro)
@@ -1,4 +1,4 @@
 <?xml version="1.0" encoding="UTF-8"?>
-<xacro:macro name="imu">
+<xacro:macro xmlns:xacro="http://www.ros.org/wiki/xacro" name="imu">
   <ros2_control name="imu" type="sensor">
     <hardware>

File: urdf/sinsei_umiusi_control/indicator_led.urdf.xacro (robot description, xacro)
@@ -1,4 +1,4 @@
 <?xml version="1.0" encoding="UTF-8"?>
-<xacro:macro name="indicator_led">
+<xacro:macro xmlns:xacro="http://www.ros.org/wiki/xacro" name="indicator_led">
   <ros2_control name="thruster_direct" type="actuator">
     <hardware>

File: urdf/sinsei_umiusi_control/raspi_camera.urdf.xacro (robot description, xacro)
@@ -1,4 +1,4 @@
 <?xml version="1.0" encoding="UTF-8"?>
-<xacro:macro name="raspi_camera">
+<xacro:macro xmlns:xacro="http://www.ros.org/wiki/xacro" name="raspi_camera">
   <ros2_control name="raspi_camera" type="actuator">
     <hardware>

File: urdf/sinsei_umiusi_control/thruster_direct.urdf.xacro (robot description, xacro)
@@ -1,4 +1,4 @@
 <?xml version="1.0" encoding="UTF-8"?>
-<xacro:macro name="thruster_direct" params="id">
+<xacro:macro xmlns:xacro="http://www.ros.org/wiki/xacro" name="thruster_direct" params="id">
   <ros2_control name="thruster_direct" type="actuator">
     <hardware>

File: urdf/sinsei_umiusi_control/usb_camera.urdf.xacro (robot description, xacro)
@@ -1,4 +1,4 @@
 <?xml version="1.0" encoding="UTF-8"?>
-<xacro:macro name="usb_camera">
+<xacro:macro xmlns:xacro="http://www.ros.org/wiki/xacro" name="usb_camera">
   <ros2_control name="usb_camera" type="actuator">
     <hardware>

Commit message: add robot tag to all xacro files

File: urdf/sinsei_umiusi_control/can.urdf.xacro (robot description, xacro)
@@ -1,44 +1,46 @@
 <?xml version="1.0" encoding="UTF-8"?>
-<xacro:macro xmlns:xacro="http://www.ros.org/wiki/xacro" name="can" params="with_thruster">
-  <ros2_control name="can" type="system">
-    <hardware>
-      <plugin>sinsei_umiusi_control/hardware/Can</plugin>
-    </hardware>
-    <xacro:if value="${with_thruster}">
-      <xacro:thruster id="1" />
-      <xacro:thruster id="2" />
-      <xacro:thruster id="3" />
-      <xacro:thruster id="4" />
-    </xacro:if>
-    <xacro:main_power />
-    <xacro:led_tape />
-  </ros2_control>
-  <!-- 内部で使うマクロ -->
-  <xacro:macro name="thruster" params="id">
-    <xacro:property name="thruster_name" value="thruster${id}" />
-    <gpio name="${thruster_name}/servo">
-      <command_interface name="thruster/enabled_raw" />
-      <command_interface name="thruster/angle_raw" />
-      <state_interface name="thruster/servo_current_raw" />
-    </gpio>
-    <gpio name="${thruster_name}/esc">
-      <command_interface name="thruster/enabled_raw" />
-      <command_interface name="thruster/thrust_raw" />
-      <state_interface name="thruster/rpm_raw" />
-    </gpio>
+<robot xmlns:xacro="http://www.ros.org/wiki/xacro" name="UMIUSI">
+  <xacro:macro name="can" params="with_thruster">
+    <ros2_control name="can" type="system">
+      <hardware>
+        <plugin>sinsei_umiusi_control/hardware/Can</plugin>
+      </hardware>
+      <xacro:if value="${with_thruster}">
+        <xacro:thruster id="1" />
+        <xacro:thruster id="2" />
+        <xacro:thruster id="3" />
+        <xacro:thruster id="4" />
+      </xacro:if>
+      <xacro:main_power />
+      <xacro:led_tape />
+    </ros2_control>
+    <!-- 内部で使うマクロ -->
+    <xacro:macro name="thruster" params="id">
+      <xacro:property name="thruster_name" value="thruster${id}" />
+      <gpio name="${thruster_name}/servo">
+        <command_interface name="thruster/enabled_raw" />
+        <command_interface name="thruster/angle_raw" />
+        <state_interface name="thruster/servo_current_raw" />
+      </gpio>
+      <gpio name="${thruster_name}/esc">
+        <command_interface name="thruster/enabled_raw" />
+        <command_interface name="thruster/thrust_raw" />
+        <state_interface name="thruster/rpm_raw" />
+      </gpio>
+    </xacro:macro>
+    <xacro:macro name="main_power">
+      <gpio name="main_power">
+        <command_interface name="main_power/enabled" />
+        <state_interface name="main_power/battery_current" />
+        <state_interface name="main_power/battery_voltage" />
+        <state_interface name="main_power/temperature" />
+        <state_interface name="main_power/water_leaked" />
+      </gpio>
+    </xacro:macro>
+    <xacro:macro name="led_tape">
+      <gpio name="led_tape">
+        <command_interface name="led_tape/color" />
+      </gpio>
+    </xacro:macro>
   </xacro:macro>
-  <xacro:macro name="main_power">
-    <gpio name="main_power">
-      <command_interface name="main_power/enabled" />
-      <state_interface name="main_power/battery_current" />
-      <state_interface name="main_power/battery_voltage" />
-      <state_interface name="main_power/temperature" />
-      <state_interface name="main_power/water_leaked" />
-    </gpio>
-  </xacro:macro>
-  <xacro:macro name="led_tape">
-    <gpio name="led_tape">
-      <command_interface name="led_tape/color" />
-    </gpio>
-  </xacro:macro>
-</xacro:macro>
+</robot>

File: urdf/sinsei_umiusi_control/headlights.urdf.xacro (robot description, xacro)
@@ -1,13 +1,15 @@
 <?xml version="1.0" encoding="UTF-8"?>
-<xacro:macro xmlns:xacro="http://www.ros.org/wiki/xacro" name="headlights">
-  <ros2_control name="headlights" type="actuator">
-    <hardware>
-      <plugin>sinsei_umiusi_control/hardware/Headlights</plugin>
-    </hardware>
-    <gpio name="headlights">
-      <command_interface name="headlights/high_beam_enabled" />
-      <command_interface name="headlights/low_beam_enabled" />
-      <command_interface name="headlights/ir_enabled" />
-    </gpio>
-  </ros2_control>
-</xacro:macro>
+<robot xmlns:xacro="http://www.ros.org/wiki/xacro" name="UMIUSI">
+  <xacro:macro name="headlights">
+    <ros2_control name="headlights" type="actuator">
+      <hardware>
+        <plugin>sinsei_umiusi_control/hardware/Headlights</plugin>
+      </hardware>
+      <gpio name="headlights">
+        <command_interface name="headlights/high_beam_enabled" />
+        <command_interface name="headlights/low_beam_enabled" />
+        <command_interface name="headlights/ir_enabled" />
+      </gpio>
+    </ros2_control>
+  </xacro:macro>
+</robot>

File: urdf/sinsei_umiusi_control/imu.urdf.xacro (robot description, xacro)
@@ -1,13 +1,15 @@
 <?xml version="1.0" encoding="UTF-8"?>
-<xacro:macro xmlns:xacro="http://www.ros.org/wiki/xacro" name="imu">
-  <ros2_control name="imu" type="sensor">
-    <hardware>
-      <plugin>sinsei_umiusi_control/hardware/Imu</plugin>
-    </hardware>
-    <gpio name="imu">
-      <state_interface name="imu/orientation" />
-      <state_interface name="imu/velocity" />
-      <state_interface name="imu/temperature" />
-    </gpio>
-  </ros2_control>
-</xacro:macro>
+<robot xmlns:xacro="http://www.ros.org/wiki/xacro" name="UMIUSI">
+  <xacro:macro name="imu">
+    <ros2_control name="imu" type="sensor">
+      <hardware>
+        <plugin>sinsei_umiusi_control/hardware/Imu</plugin>
+      </hardware>
+      <gpio name="imu">
+        <state_interface name="imu/orientation" />
+        <state_interface name="imu/velocity" />
+        <state_interface name="imu/temperature" />
+      </gpio>
+    </ros2_control>
+  </xacro:macro>
+</robot>

File: urdf/sinsei_umiusi_control/indicator_led.urdf.xacro (robot description, xacro)
@@ -1,11 +1,13 @@
 <?xml version="1.0" encoding="UTF-8"?>
-<xacro:macro xmlns:xacro="http://www.ros.org/wiki/xacro" name="indicator_led">
-  <ros2_control name="thruster_direct" type="actuator">
-    <hardware>
-      <plugin>sinsei_umiusi_control/hardware/IndicatorLed</plugin>
-    </hardware>
-    <gpio name="indicator_led">
-      <command_interface name="indicator_led/enabled" />
-    </gpio>
-  </ros2_control>
-</xacro:macro>
+<robot xmlns:xacro="http://www.ros.org/wiki/xacro" name="UMIUSI">
+  <xacro:macro name="indicator_led">
+    <ros2_control name="thruster_direct" type="actuator">
+      <hardware>
+        <plugin>sinsei_umiusi_control/hardware/IndicatorLed</plugin>
+      </hardware>
+      <gpio name="indicator_led">
+        <command_interface name="indicator_led/enabled" />
+      </gpio>
+    </ros2_control>
+  </xacro:macro>
+</robot>

File: urdf/sinsei_umiusi_control/raspi_camera.urdf.xacro (robot description, xacro)
@@ -1,12 +1,14 @@
 <?xml version="1.0" encoding="UTF-8"?>
-<xacro:macro xmlns:xacro="http://www.ros.org/wiki/xacro" name="raspi_camera">
-  <ros2_control name="raspi_camera" type="actuator">
-    <hardware>
-      <plugin>sinsei_umiusi_control/hardware/RaspiCamera</plugin>
-    </hardware>
-    <gpio name="raspi_camera">
-      <command_interface name="raspi_camera/config" />
-      <state_interface name="raspi_camera/image" />
-    </gpio>
-  </ros2_control>
-</xacro:macro>
+<robot xmlns:xacro="http://www.ros.org/wiki/xacro" name="UMIUSI">
+  <xacro:macro name="raspi_camera">
+    <ros2_control name="raspi_camera" type="actuator">
+      <hardware>
+        <plugin>sinsei_umiusi_control/hardware/RaspiCamera</plugin>
+      </hardware>
+      <gpio name="raspi_camera">
+        <command_interface name="raspi_camera/config" />
+        <state_interface name="raspi_camera/image" />
+      </gpio>
+    </ros2_control>
+  </xacro:macro>
+</robot>

File: urdf/sinsei_umiusi_control/thruster_direct.urdf.xacro (robot description, xacro)
@@ -1,24 +1,26 @@
 <?xml version="1.0" encoding="UTF-8"?>
-<xacro:macro xmlns:xacro="http://www.ros.org/wiki/xacro" name="thruster_direct" params="id">
-  <ros2_control name="thruster_direct" type="actuator">
-    <hardware>
-      <plugin>sinsei_umiusi_control/hardware/ThrusterDirect</plugin>
-    </hardware>
-    <xacro:thruster_direct id="1" />
-    <xacro:thruster_direct id="2" />
-    <xacro:thruster_direct id="3" />
-    <xacro:thruster_direct id="4" />
-  </ros2_control>
-  <!-- 内部で使うマクロ -->
-  <xacro:macro name="thruster_direct" params="id">
-    <xacro:property name="thruster_name" value="thruster_direct${id}" />
-    <gpio name="${thruster_name}/servo_direct">
-      <command_interface name="thruster_direct/enabled_raw" />
-      <command_interface name="thruster_direct/angle_raw" />
-    </gpio>
-    <gpio name="${thruster_name}/esc_direct">
-      <command_interface name="thruster_direct/enabled_raw" />
-      <command_interface name="thruster_direct/thrust_raw" />
-    </gpio>
+<robot xmlns:xacro="http://www.ros.org/wiki/xacro" name="UMIUSI">
+  <xacro:macro name="thruster_direct">
+    <ros2_control name="thruster_direct" type="actuator">
+      <hardware>
+        <plugin>sinsei_umiusi_control/hardware/ThrusterDirect</plugin>
+      </hardware>
+      <xacro:thruster_direct id="1" />
+      <xacro:thruster_direct id="2" />
+      <xacro:thruster_direct id="3" />
+      <xacro:thruster_direct id="4" />
+    </ros2_control>
+    <!-- 内部で使うマクロ -->
+    <xacro:macro name="thruster_direct" params="id">
+      <xacro:property name="thruster_name" value="thruster_direct${id}" />
+      <gpio name="${thruster_name}/servo_direct">
+        <command_interface name="thruster_direct/enabled_raw" />
+        <command_interface name="thruster_direct/angle_raw" />
+      </gpio>
+      <gpio name="${thruster_name}/esc_direct">
+        <command_interface name="thruster_direct/enabled_raw" />
+        <command_interface name="thruster_direct/thrust_raw" />
+      </gpio>
+    </xacro:macro>
   </xacro:macro>
-</xacro:macro>
+</robot>

File: urdf/sinsei_umiusi_control/usb_camera.urdf.xacro (robot description, xacro)
@@ -1,12 +1,14 @@
 <?xml version="1.0" encoding="UTF-8"?>
-<xacro:macro xmlns:xacro="http://www.ros.org/wiki/xacro" name="usb_camera">
-  <ros2_control name="usb_camera" type="actuator">
-    <hardware>
-      <plugin>sinsei_umiusi_control/hardware/UsbCamera</plugin>
-    </hardware>
-    <gpio name="usb_camera">
-      <command_interface name="usb_camera/config" />
-      <state_interface name="usb_camera/image" />
-    </gpio>
-  </ros2_control>
-</xacro:macro>
+<robot xmlns:xacro="http://www.ros.org/wiki/xacro" name="UMIUSI">
+  <xacro:macro name="usb_camera">
+    <ros2_control name="usb_camera" type="actuator">
+      <hardware>
+        <plugin>sinsei_umiusi_control/hardware/UsbCamera</plugin>
+      </hardware>
+      <gpio name="usb_camera">
+        <command_interface name="usb_camera/config" />
+        <state_interface name="usb_camera/image" />
+      </gpio>
+    </ros2_control>
+  </xacro:macro>
+</robot>
