Commit message: feat(alexandrite): SteppingMotorDriver基板でバラストを動かせるようにする
SteppingMotorDriver基板1枚の2軸（M1/M2）で動かすバラストを、暫定的にtopicから
操作できるようにする。

- can::SteppingMotorDriverModel: 0x311/0x312の送信と0x318/0x319の受信に対応
- hardware::Can: ballast1/ballast2のインターフェースを追加（Alexandriteのみ）
  - 準備完了前の目標は基板に無視されるため、同じ目標も定期的に送り直す
  - ゼロ点の取り直しは要求回数が増えたときだけ行う
- BallastController: std_msgsのtopicで目標・ゼロ点取り直しを受け付け、位置・状態を公開
- CAN周りのファイルにclang-formatを適用

Co-Authored-By: Claude Opus 5.5 <noreply@anthropic.com>

File: urdf/sinsei_umiusi_control/can.urdf.xacro (robot description, xacro)
@@ -36,4 +36,34 @@
         </command_interface>
       </xacro:if>
+    </gpio>
+  </xacro:macro>
+  <!-- SteppingMotorDriver基板の1軸で動かすバラスト。axisは0 = M1、1 = M2 -->
+  <xacro:macro name="stepping_motor_ballast" params="name axis">
+    <gpio name="${name}">
+      <param name="stepping_motor_driver_axis">${axis}</param>
+      <command_interface name="target" data_type="double">
+        <!-- 行程に対する割合（0.0〜1.0）。負の値かNaNの間は送らない（初期値にNaNは使えない） -->
+        <param name="initial_value">-1.0</param>
+      </command_interface>
+      <command_interface name="calibrate" data_type="double">
+        <!-- 値が変わるたびにゼロ点を取り直す -->
+        <param name="initial_value">0.0</param>
+      </command_interface>
+      <state_interface name="position" data_type="double">
+        <param name="initial_value">0.0</param>
+      </state_interface>
+      <state_interface name="state" data_type="double">
+        <param name="initial_value">0.0</param>
+      </state_interface>
+      <state_interface name="fault_reason" data_type="double">
+        <param name="initial_value">0.0</param>
+      </state_interface>
+      <state_interface name="flags" data_type="double">
+        <param name="initial_value">0.0</param>
+      </state_interface>
+      <state_interface name="health" data_type="double">
+        <!-- false (Cannot use bool type due to ros2_control bug) -->
+        <param name="initial_value">0.0</param>
+      </state_interface>
     </gpio>
   </xacro:macro>
@@ -128,4 +158,6 @@
       <xacro:vesc_actuator name="crawler_left" vesc_id="${crawler_left_vesc_id}" motor_type="dc" has_servo="false" />
       <xacro:vesc_actuator name="crawler_right" vesc_id="${crawler_right_vesc_id}" motor_type="dc" has_servo="false" />
+      <xacro:stepping_motor_ballast name="ballast1" axis="0" />
+      <xacro:stepping_motor_ballast name="ballast2" axis="1" />
       <xacro:can_auxiliary_interfaces />
     </ros2_control>
