Commit message: refactor(hardware): use `thruster_direct` class for each thrusters

File: urdf/sinsei_umiusi_control/thruster_direct.urdf.xacro (robot description, xacro)
@@ -2,10 +2,10 @@
 <robot xmlns:xacro="http://www.ros.org/wiki/xacro" name="UMIUSI">
   <xacro:macro name="thruster_direct">
-    <ros2_control name="thruster_direct" type="actuator">
-      <hardware>
-        <plugin>sinsei_umiusi_control/hardware/ThrusterDirect</plugin>
-      </hardware>
-      <xacro:macro name="thruster_direct" params="id">
-        <xacro:property name="thruster_name" value="thruster_direct${id}" />
+    <xacro:macro name="thruster_direct" params="id">
+      <xacro:property name="thruster_name" value="thruster_direct${id}" />
+      <ros2_control name="${thruster_name}" type="actuator">
+        <hardware>
+          <plugin>sinsei_umiusi_control/hardware/ThrusterDirect</plugin>
+        </hardware>
         <gpio name="${thruster_name}/servo_direct">
           <command_interface name="thruster_direct/enabled_raw" />
@@ -16,10 +16,10 @@
           <command_interface name="thruster_direct/thrust_raw" />
         </gpio>
-      </xacro:macro>
-      <xacro:thruster_direct id="1" />
-      <xacro:thruster_direct id="2" />
-      <xacro:thruster_direct id="3" />
-      <xacro:thruster_direct id="4" />
-    </ros2_control>
+      </ros2_control>
+    </xacro:macro>
+    <xacro:thruster_direct id="1" />
+    <xacro:thruster_direct id="2" />
+    <xacro:thruster_direct id="3" />
+    <xacro:thruster_direct id="4" />
   </xacro:macro>
 </robot>
