Commit message: correct wrong xacro syntax

File: urdf/sinsei_umiusi_control.urdf.xacro (robot description, xacro)
@@ -1,5 +1,5 @@
 <?xml version="1.0" encoding="UTF-8"?>
 <robot xmlns:xacro="http://www.ros.org/wiki/xacro" name="UMIUSI">
-  <xacro:arg name="thruster_mode" default="can" />
+  <xacro:arg name="thruster_mode" default="'can'" />
   <xacro:include filename="sinsei_umiusi_control/can.urdf.xacro" />
   <xacro:include filename="sinsei_umiusi_control/thruster_direct.urdf.xacro" />

File: urdf/sinsei_umiusi_control/can.urdf.xacro (robot description, xacro)
@@ -6,4 +6,17 @@
         <plugin>sinsei_umiusi_control/hardware/Can</plugin>
       </hardware>
+      <xacro:macro name="thruster" params="id">
+        <xacro:property name="thruster_name" value="thruster${id}" />
+        <gpio name="${thruster_name}/servo">
+          <command_interface name="thruster/enabled_raw" />
+          <command_interface name="thruster/angle_raw" />
+          <state_interface name="thruster/servo_current_raw" />
+        </gpio>
+        <gpio name="${thruster_name}/esc">
+          <command_interface name="thruster/enabled_raw" />
+          <command_interface name="thruster/thrust_raw" />
+          <state_interface name="thruster/rpm_raw" />
+        </gpio>
+      </xacro:macro>
       <xacro:if value="${with_thruster}">
         <xacro:thruster id="1" />
@@ -12,22 +25,4 @@
         <xacro:thruster id="4" />
       </xacro:if>
-      <xacro:main_power />
-      <xacro:led_tape />
-    </ros2_control>
-    <!-- 内部で使うマクロ -->
-    <xacro:macro name="thruster" params="id">
-      <xacro:property name="thruster_name" value="thruster${id}" />
-      <gpio name="${thruster_name}/servo">
-        <command_interface name="thruster/enabled_raw" />
-        <command_interface name="thruster/angle_raw" />
-        <state_interface name="thruster/servo_current_raw" />
-      </gpio>
-      <gpio name="${thruster_name}/esc">
-        <command_interface name="thruster/enabled_raw" />
-        <command_interface name="thruster/thrust_raw" />
-        <state_interface name="thruster/rpm_raw" />
-      </gpio>
-    </xacro:macro>
-    <xacro:macro name="main_power">
       <gpio name="main_power">
         <command_interface name="main_power/enabled" />
@@ -37,10 +32,8 @@
         <state_interface name="main_power/water_leaked" />
       </gpio>
-    </xacro:macro>
-    <xacro:macro name="led_tape">
       <gpio name="led_tape">
         <command_interface name="led_tape/color" />
       </gpio>
-    </xacro:macro>
+    </ros2_control>
   </xacro:macro>
 </robot>

File: urdf/sinsei_umiusi_control/thruster_direct.urdf.xacro (robot description, xacro)
@@ -6,4 +6,15 @@
         <plugin>sinsei_umiusi_control/hardware/ThrusterDirect</plugin>
       </hardware>
+      <xacro:macro name="thruster_direct" params="id">
+        <xacro:property name="thruster_name" value="thruster_direct${id}" />
+        <gpio name="${thruster_name}/servo_direct">
+          <command_interface name="thruster_direct/enabled_raw" />
+          <command_interface name="thruster_direct/angle_raw" />
+        </gpio>
+        <gpio name="${thruster_name}/esc_direct">
+          <command_interface name="thruster_direct/enabled_raw" />
+          <command_interface name="thruster_direct/thrust_raw" />
+        </gpio>
+      </xacro:macro>
       <xacro:thruster_direct id="1" />
       <xacro:thruster_direct id="2" />
@@ -11,16 +22,4 @@
       <xacro:thruster_direct id="4" />
     </ros2_control>
-    <!-- 内部で使うマクロ -->
-    <xacro:macro name="thruster_direct" params="id">
-      <xacro:property name="thruster_name" value="thruster_direct${id}" />
-      <gpio name="${thruster_name}/servo_direct">
-        <command_interface name="thruster_direct/enabled_raw" />
-        <command_interface name="thruster_direct/angle_raw" />
-      </gpio>
-      <gpio name="${thruster_name}/esc_direct">
-        <command_interface name="thruster_direct/enabled_raw" />
-        <command_interface name="thruster_direct/thrust_raw" />
-      </gpio>
-    </xacro:macro>
   </xacro:macro>
 </robot>

Commit message: fix(urdf): add link

File: urdf/sinsei_umiusi_control.urdf.xacro (robot description, xacro)
@@ -9,4 +9,5 @@
   <xacro:include filename="sinsei_umiusi_control/usb_camera.urdf.xacro" />
   <xacro:include filename="sinsei_umiusi_control/raspi_camera.urdf.xacro" />
+  <link name="base_link"></link>
   <xacro:if value="${$(arg thruster_mode) == 'can'}">
     <xacro:can with_thruster="true" />

Commit message: refactor(urdf): :recycle: refactor robot descriptions

File: urdf/sinsei_umiusi_control.urdf.xacro (robot description, xacro)
@@ -1,17 +1,31 @@
 <?xml version="1.0" encoding="UTF-8"?>
 <robot xmlns:xacro="http://www.ros.org/wiki/xacro" name="UMIUSI">
-  <xacro:arg name="thruster_mode" default="'unknown'" />
-  <xacro:include filename="sinsei_umiusi_control/can.urdf.xacro" />
-  <xacro:include filename="sinsei_umiusi_control/thruster_direct.urdf.xacro" />
-  <xacro:include filename="sinsei_umiusi_control/indicator_led.urdf.xacro" />
-  <xacro:include filename="sinsei_umiusi_control/imu.urdf.xacro" />
-  <xacro:include filename="sinsei_umiusi_control/headlights.urdf.xacro" />
-  <link name="base_link"></link>
-  <xacro:can thruster_mode="$(arg thruster_mode)" />
-  <xacro:if value="${$(arg thruster_mode) == 'direct'}">
-    <xacro:thruster_direct />
-  </xacro:if>
-  <xacro:indicator_led />
-  <xacro:imu />
-  <xacro:headlights />
+  <xacro:macro name="sinsei_umiusi_control"
+    params="
+      thruster_mode
+      high_beam_pin
+      low_beam_pin
+      ir_pin
+      indicator_led_pin
+      mock
+    ">
+    <xacro:include filename="sinsei_umiusi_control/can.urdf.xacro" />
+    <xacro:include filename="sinsei_umiusi_control/thruster_direct.urdf.xacro" />
+    <xacro:include filename="sinsei_umiusi_control/indicator_led.urdf.xacro" />
+    <xacro:include filename="sinsei_umiusi_control/imu.urdf.xacro" />
+    <xacro:include filename="sinsei_umiusi_control/headlights.urdf.xacro" />
+    <link name="base_link"></link>
+    <xacro:can thruster_mode="${thruster_mode}" />
+    <xacro:if value="${thruster_mode == 'direct'}">
+      <xacro:thruster_direct />
+    </xacro:if>
+    <xacro:imu />
+    <xacro:headlights
+      high_beam_pin="${high_beam_pin}"
+      low_beam_pin="${low_beam_pin}"
+      ir_pin="${ir_pin}" />
+    <xacro:indicator_led
+      pin="${indicator_led_pin}"
+    />
+  </xacro:macro>
 </robot>

File: urdf/sinsei_umiusi_control/headlights.urdf.xacro (robot description, xacro)
@@ -1,8 +1,11 @@
 <?xml version="1.0" encoding="UTF-8"?>
 <robot xmlns:xacro="http://www.ros.org/wiki/xacro" name="UMIUSI">
-  <xacro:macro name="headlights">
+  <xacro:macro name="headlights" params="high_beam_pin low_beam_pin ir_pin">
     <ros2_control name="headlights" type="system">
       <hardware>
         <plugin>sinsei_umiusi_control/hardware/Headlights</plugin>
+        <param name="high_beam_pin">${high_beam_pin}</param>
+        <param name="low_beam_pin">${low_beam_pin}</param>
+        <param name="ir_pin">${ir_pin}</param>
       </hardware>
       <gpio name="headlights">

File: urdf/sinsei_umiusi_control/indicator_led.urdf.xacro (robot description, xacro)
@@ -1,8 +1,9 @@
 <?xml version="1.0" encoding="UTF-8"?>
 <robot xmlns:xacro="http://www.ros.org/wiki/xacro" name="UMIUSI">
-  <xacro:macro name="indicator_led">
+  <xacro:macro name="indicator_led" params="pin">
     <ros2_control name="indicator_led" type="system">
       <hardware>
         <plugin>sinsei_umiusi_control/hardware/IndicatorLed</plugin>
+        <param name="pin">${pin}</param>
       </hardware>
       <gpio name="indicator_led">
