Commit message: fix(urdf): :adhesive_bandage: move link declaration to main.urdf.xacro

File: urdf/main.urdf.xacro (robot description, xacro)
@@ -7,4 +7,5 @@
   <xacro:arg name="indicator_led_pin" default="'unknown'" />
   <xacro:include filename="sinsei_umiusi_control.urdf.xacro" />
+  <link name="base_link"></link>
   <xacro:sinsei_umiusi_control
     thruster_mode="$(arg thruster_mode)"

File: urdf/sinsei_umiusi_control.urdf.xacro (robot description, xacro)
@@ -15,5 +15,4 @@
     <xacro:include filename="sinsei_umiusi_control/imu.urdf.xacro" />
     <xacro:include filename="sinsei_umiusi_control/headlights.urdf.xacro" />
-    <link name="base_link"></link>
     <xacro:can thruster_mode="${thruster_mode}" />
     <xacro:if value="${thruster_mode == 'direct'}">

Commit message: feat(can): VESCのIDをLaunch argumentとして指定

File: urdf/main.urdf.xacro (robot description, xacro)
@@ -6,4 +6,8 @@
   <xacro:arg name="ir_pin" default="'unknown'" />
   <xacro:arg name="indicator_led_pin" default="'unknown'" />
+  <xacro:arg name="vesc1_id" default="'unknown'" />
+  <xacro:arg name="vesc2_id" default="'unknown'" />
+  <xacro:arg name="vesc3_id" default="'unknown'" />
+  <xacro:arg name="vesc4_id" default="'unknown'" />
   <xacro:include filename="sinsei_umiusi_control.urdf.xacro" />
   <link name="base_link"></link>
@@ -14,4 +18,8 @@
     ir_pin="$(arg ir_pin)"
     indicator_led_pin="$(arg indicator_led_pin)"
+    vesc1_id="$(arg vesc1_id)"
+    vesc2_id="$(arg vesc2_id)"
+    vesc3_id="$(arg vesc3_id)"
+    vesc4_id="$(arg vesc4_id)"
     mock="false"
   />

File: urdf/sinsei_umiusi_control.urdf.xacro (robot description, xacro)
@@ -8,4 +8,8 @@
       ir_pin
       indicator_led_pin
+      vesc1_id
+      vesc2_id
+      vesc3_id
+      vesc4_id
       mock
     ">
@@ -15,5 +19,11 @@
     <xacro:include filename="sinsei_umiusi_control/imu.urdf.xacro" />
     <xacro:include filename="sinsei_umiusi_control/headlights.urdf.xacro" />
-    <xacro:can thruster_mode="${thruster_mode}" />
+    <xacro:can
+      thruster_mode="${thruster_mode}"
+      vesc1_id="${vesc1_id}"
+      vesc2_id="${vesc2_id}"
+      vesc3_id="${vesc3_id}"
+      vesc4_id="${vesc4_id}"
+    />
     <xacro:if value="${thruster_mode == 'direct'}">
       <xacro:thruster_direct />

File: urdf/sinsei_umiusi_control/can.urdf.xacro (robot description, xacro)
@@ -1,9 +1,13 @@
 <?xml version="1.0" encoding="UTF-8"?>
 <robot xmlns:xacro="http://www.ros.org/wiki/xacro" name="UMIUSI">
-  <xacro:macro name="can" params="thruster_mode">
+  <xacro:macro name="can" params="thruster_mode vesc1_id vesc2_id vesc3_id vesc4_id">
     <ros2_control name="can" type="system">
       <hardware>
         <plugin>sinsei_umiusi_control/hardware/Can</plugin>
         <param name="thruster_mode">${thruster_mode}</param>
+        <param name="vesc1_id">${vesc1_id}</param>
+        <param name="vesc2_id">${vesc2_id}</param>
+        <param name="vesc3_id">${vesc3_id}</param>
+        <param name="vesc4_id">${vesc4_id}</param>
       </hardware>
       <xacro:macro name="thruster" params="id">

Commit message: :sparkles: LEDテープの制御周期をパラメータ化

File: urdf/main.urdf.xacro (robot description, xacro)
@@ -10,4 +10,5 @@
   <xacro:arg name="vesc3_id" default="'unknown'" />
   <xacro:arg name="vesc4_id" default="'unknown'" />
+  <xacro:arg name="period_led_tape_per_thrusters" default="'unknown'" />
   <xacro:include filename="sinsei_umiusi_control.urdf.xacro" />
   <link name="base_link"></link>
@@ -22,4 +23,5 @@
     vesc3_id="$(arg vesc3_id)"
     vesc4_id="$(arg vesc4_id)"
+    period_led_tape_per_thrusters="$(arg period_led_tape_per_thrusters)"
     mock="false"
   />

File: urdf/sinsei_umiusi_control.urdf.xacro (robot description, xacro)
@@ -12,4 +12,5 @@
       vesc3_id
       vesc4_id
+      period_led_tape_per_thrusters
       mock
     ">
@@ -25,4 +26,5 @@
       vesc3_id="${vesc3_id}"
       vesc4_id="${vesc4_id}"
+      period_led_tape_per_thrusters="${period_led_tape_per_thrusters}"
     />
     <xacro:if value="${thruster_mode == 'direct'}">

File: urdf/sinsei_umiusi_control/can.urdf.xacro (robot description, xacro)
@@ -1,5 +1,6 @@
 <?xml version="1.0" encoding="UTF-8"?>
 <robot xmlns:xacro="http://www.ros.org/wiki/xacro" name="UMIUSI">
-  <xacro:macro name="can" params="thruster_mode vesc1_id vesc2_id vesc3_id vesc4_id">
+  <xacro:macro name="can"
+    params="thruster_mode vesc1_id vesc2_id vesc3_id vesc4_id period_led_tape_per_thrusters">
     <ros2_control name="can" type="system">
       <hardware>
@@ -10,4 +11,5 @@
         <param name="vesc3_id">${vesc3_id}</param>
         <param name="vesc4_id">${vesc4_id}</param>
+        <param name="period_led_tape_per_thrusters">${period_led_tape_per_thrusters}</param>
       </hardware>
       <xacro:macro name="thruster" params="id">

Commit message: feat(thruster_direct): Hardware Componentを実装

File: urdf/main.urdf.xacro (robot description, xacro)
@@ -6,4 +6,12 @@
   <xacro:arg name="ir_pin" default="'unknown'" />
   <xacro:arg name="indicator_led_pin" default="'unknown'" />
+  <xacro:arg name="servo_direct1_pin" default="'unknown'" />
+  <xacro:arg name="servo_direct2_pin" default="'unknown'" />
+  <xacro:arg name="servo_direct3_pin" default="'unknown'" />
+  <xacro:arg name="servo_direct4_pin" default="'unknown'" />
+  <xacro:arg name="esc_direct1_pin" default="'unknown'" />
+  <xacro:arg name="esc_direct2_pin" default="'unknown'" />
+  <xacro:arg name="esc_direct3_pin" default="'unknown'" />
+  <xacro:arg name="esc_direct4_pin" default="'unknown'" />
   <xacro:arg name="vesc1_id" default="'unknown'" />
   <xacro:arg name="vesc2_id" default="'unknown'" />
@@ -19,4 +27,12 @@
     ir_pin="$(arg ir_pin)"
     indicator_led_pin="$(arg indicator_led_pin)"
+    servo_direct1_pin="$(arg servo_direct1_pin)"
+    servo_direct2_pin="$(arg servo_direct2_pin)"
+    servo_direct3_pin="$(arg servo_direct3_pin)"
+    servo_direct4_pin="$(arg servo_direct4_pin)"
+    esc_direct1_pin="$(arg esc_direct1_pin)"
+    esc_direct2_pin="$(arg esc_direct2_pin)"
+    esc_direct3_pin="$(arg esc_direct3_pin)"
+    esc_direct4_pin="$(arg esc_direct4_pin)"
     vesc1_id="$(arg vesc1_id)"
     vesc2_id="$(arg vesc2_id)"

File: urdf/sinsei_umiusi_control.urdf.xacro (robot description, xacro)
@@ -8,4 +8,12 @@
       ir_pin
       indicator_led_pin
+      servo_direct1_pin
+      servo_direct2_pin
+      servo_direct3_pin
+      servo_direct4_pin
+      esc_direct1_pin
+      esc_direct2_pin
+      esc_direct3_pin
+      esc_direct4_pin
       vesc1_id
       vesc2_id
@@ -29,5 +37,14 @@
     />
     <xacro:if value="${thruster_mode == 'direct'}">
-      <xacro:thruster_direct />
+      <xacro:thruster_direct
+        servo1_pin="${servo_direct1_pin}"
+        servo2_pin="${servo_direct2_pin}"
+        servo3_pin="${servo_direct3_pin}"
+        servo4_pin="${servo_direct4_pin}"
+        esc1_pin="${esc_direct1_pin}"
+        esc2_pin="${esc_direct2_pin}"
+        esc3_pin="${esc_direct3_pin}"
+        esc4_pin="${esc_direct4_pin}"
+      />
     </xacro:if>
     <xacro:imu />

File: urdf/sinsei_umiusi_control/thruster_direct.urdf.xacro (robot description, xacro)
@@ -1,15 +1,18 @@
 <?xml version="1.0" encoding="UTF-8"?>
 <robot xmlns:xacro="http://www.ros.org/wiki/xacro" name="UMIUSI">
-  <xacro:macro name="thruster_direct">
-    <xacro:macro name="thruster_direct" params="id">
+  <xacro:macro name="thruster_direct"
+    params="servo1_pin servo2_pin servo3_pin servo4_pin esc1_pin esc2_pin esc3_pin esc4_pin">
+    <xacro:macro name="thruster_direct" params="id servo_pin esc_pin">
       <xacro:property name="thruster_name" value="thruster_direct${id}" />
       <ros2_control name="${thruster_name}/servo" type="system">
         <hardware>
           <plugin>sinsei_umiusi_control/hardware/ServoDirect</plugin>
+          <param name="id">${id}</param>
+          <param name="pin">${servo_pin}</param>
         </hardware>
         <gpio name="${thruster_name}/servo">
           <command_interface name="enabled" />
           <command_interface name="angle" />
-          <state_interface name="state" />
+          <state_interface name="health" />
         </gpio>
       </ros2_control>
@@ -17,4 +20,6 @@
         <hardware>
           <plugin>sinsei_umiusi_control/hardware/EscDirect</plugin>
+          <param name="id">${id}</param>
+          <param name="pin">${esc_pin}</param>
         </hardware>
         <gpio name="${thruster_name}/esc">
@@ -25,8 +30,8 @@
       </ros2_control>
     </xacro:macro>
-    <xacro:thruster_direct id="1" />
-    <xacro:thruster_direct id="2" />
-    <xacro:thruster_direct id="3" />
-    <xacro:thruster_direct id="4" />
+    <xacro:thruster_direct id="1" servo_pin="${servo1_pin}" esc_pin="${esc1_pin}" />
+    <xacro:thruster_direct id="2" servo_pin="${servo2_pin}" esc_pin="${esc2_pin}" />
+    <xacro:thruster_direct id="3" servo_pin="${servo3_pin}" esc_pin="${esc3_pin}" />
+    <xacro:thruster_direct id="4" servo_pin="${servo4_pin}" esc_pin="${esc4_pin}" />
   </xacro:macro>
 </robot>

Commit message: feat(direct): サーボのパルス幅の上限/下限をパラメーター化

File: urdf/main.urdf.xacro (robot description, xacro)
@@ -6,4 +6,12 @@
   <xacro:arg name="ir_pin" default="'unknown'" />
   <xacro:arg name="indicator_led_pin" default="'unknown'" />
+  <xacro:arg name="servo_direct1_min_pulse_width" default="'unknown'" />
+  <xacro:arg name="servo_direct1_max_pulse_width" default="'unknown'" />
+  <xacro:arg name="servo_direct2_min_pulse_width" default="'unknown'" />
+  <xacro:arg name="servo_direct2_max_pulse_width" default="'unknown'" />
+  <xacro:arg name="servo_direct3_min_pulse_width" default="'unknown'" />
+  <xacro:arg name="servo_direct3_max_pulse_width" default="'unknown'" />
+  <xacro:arg name="servo_direct4_min_pulse_width" default="'unknown'" />
+  <xacro:arg name="servo_direct4_max_pulse_width" default="'unknown'" />
   <xacro:arg name="servo_direct1_pin" default="'unknown'" />
   <xacro:arg name="servo_direct2_pin" default="'unknown'" />
@@ -27,4 +35,12 @@
     ir_pin="$(arg ir_pin)"
     indicator_led_pin="$(arg indicator_led_pin)"
+    servo_direct1_min_pulse_width="$(arg servo_direct1_min_pulse_width)"
+    servo_direct1_max_pulse_width="$(arg servo_direct1_max_pulse_width)"
+    servo_direct2_min_pulse_width="$(arg servo_direct2_min_pulse_width)"
+    servo_direct2_max_pulse_width="$(arg servo_direct2_max_pulse_width)"
+    servo_direct3_min_pulse_width="$(arg servo_direct3_min_pulse_width)"
+    servo_direct3_max_pulse_width="$(arg servo_direct3_max_pulse_width)"
+    servo_direct4_min_pulse_width="$(arg servo_direct4_min_pulse_width)"
+    servo_direct4_max_pulse_width="$(arg servo_direct4_max_pulse_width)"
     servo_direct1_pin="$(arg servo_direct1_pin)"
     servo_direct2_pin="$(arg servo_direct2_pin)"

File: urdf/sinsei_umiusi_control.urdf.xacro (robot description, xacro)
@@ -8,4 +8,12 @@
       ir_pin
       indicator_led_pin
+      servo_direct1_min_pulse_width
+      servo_direct1_max_pulse_width
+      servo_direct2_min_pulse_width
+      servo_direct2_max_pulse_width
+      servo_direct3_min_pulse_width
+      servo_direct3_max_pulse_width
+      servo_direct4_min_pulse_width
+      servo_direct4_max_pulse_width
       servo_direct1_pin
       servo_direct2_pin
@@ -38,4 +46,12 @@
     <xacro:if value="${thruster_mode == 'direct'}">
       <xacro:thruster_direct
+        servo1_min_pulse_width="${servo_direct1_min_pulse_width}"
+        servo1_max_pulse_width="${servo_direct1_max_pulse_width}"
+        servo2_min_pulse_width="${servo_direct2_min_pulse_width}"
+        servo2_max_pulse_width="${servo_direct2_max_pulse_width}"
+        servo3_min_pulse_width="${servo_direct3_min_pulse_width}"
+        servo3_max_pulse_width="${servo_direct3_max_pulse_width}"
+        servo4_min_pulse_width="${servo_direct4_min_pulse_width}"
+        servo4_max_pulse_width="${servo_direct4_max_pulse_width}"
         servo1_pin="${servo_direct1_pin}"
         servo2_pin="${servo_direct2_pin}"

File: urdf/sinsei_umiusi_control/thruster_direct.urdf.xacro (robot description, xacro)
@@ -2,6 +2,13 @@
 <robot xmlns:xacro="http://www.ros.org/wiki/xacro" name="UMIUSI">
   <xacro:macro name="thruster_direct"
-    params="servo1_pin servo2_pin servo3_pin servo4_pin esc1_pin esc2_pin esc3_pin esc4_pin">
-    <xacro:macro name="thruster_direct" params="id servo_pin esc_pin">
+    params="
+    servo1_min_pulse_width servo1_max_pulse_width
+    servo2_min_pulse_width servo2_max_pulse_width
+    servo3_min_pulse_width servo3_max_pulse_width
+    servo4_min_pulse_width servo4_max_pulse_width
+    servo1_pin servo2_pin servo3_pin servo4_pin
+    esc1_pin esc2_pin esc3_pin esc4_pin">
+    <xacro:macro name="thruster_direct"
+      params="id servo_min_pulse_width servo_max_pulse_width servo_pin esc_pin">
       <xacro:property name="thruster_name" value="thruster_direct${id}" />
       <ros2_control name="${thruster_name}/servo" type="system">
@@ -10,4 +17,6 @@
           <param name="id">${id}</param>
           <param name="pin">${servo_pin}</param>
+          <param name="min_pulse_width">${servo_min_pulse_width}</param>
+          <param name="max_pulse_width">${servo_max_pulse_width}</param>
         </hardware>
         <gpio name="${thruster_name}/servo">
@@ -30,8 +39,16 @@
       </ros2_control>
     </xacro:macro>
-    <xacro:thruster_direct id="1" servo_pin="${servo1_pin}" esc_pin="${esc1_pin}" />
-    <xacro:thruster_direct id="2" servo_pin="${servo2_pin}" esc_pin="${esc2_pin}" />
-    <xacro:thruster_direct id="3" servo_pin="${servo3_pin}" esc_pin="${esc3_pin}" />
-    <xacro:thruster_direct id="4" servo_pin="${servo4_pin}" esc_pin="${esc4_pin}" />
+    <xacro:thruster_direct id="1" servo_min_pulse_width="${servo1_min_pulse_width}"
+      servo_max_pulse_width="${servo1_max_pulse_width}" servo_pin="${servo1_pin}"
+      esc_pin="${esc1_pin}" />
+    <xacro:thruster_direct id="2" servo_min_pulse_width="${servo2_min_pulse_width}"
+      servo_max_pulse_width="${servo2_max_pulse_width}" servo_pin="${servo2_pin}"
+      esc_pin="${esc2_pin}" />
+    <xacro:thruster_direct id="3" servo_min_pulse_width="${servo3_min_pulse_width}"
+      servo_max_pulse_width="${servo3_max_pulse_width}" servo_pin="${servo3_pin}"
+      esc_pin="${esc3_pin}" />
+    <xacro:thruster_direct id="4" servo_min_pulse_width="${servo4_min_pulse_width}"
+      servo_max_pulse_width="${servo4_max_pulse_width}" servo_pin="${servo4_pin}"
+      esc_pin="${esc4_pin}" />
   </xacro:macro>
 </robot>

Commit message: feat(gpio): pigpiod -> libgpiodに移行

File: urdf/main.urdf.xacro (robot description, xacro)
@@ -1,8 +1,9 @@
 <?xml version="1.0" encoding="UTF-8"?>
 <robot xmlns:xacro="http://www.ros.org/wiki/xacro" name="UMIUSI">
-  <xacro:arg name="high_beam_pin" default="'unknown'" />
-  <xacro:arg name="low_beam_pin" default="'unknown'" />
-  <xacro:arg name="ir_pin" default="'unknown'" />
-  <xacro:arg name="indicator_led_pin" default="'unknown'" />
+  <xacro:arg name="gpiochip_device" default="'unknown'" />
+  <xacro:arg name="high_beam_line_offset" default="'unknown'" />
+  <xacro:arg name="low_beam_line_offset" default="'unknown'" />
+  <xacro:arg name="ir_line_offset" default="'unknown'" />
+  <xacro:arg name="indicator_led_line_offset" default="'unknown'" />
   <xacro:arg name="vesc1_id" default="'unknown'" />
   <xacro:arg name="vesc2_id" default="'unknown'" />
@@ -14,8 +15,9 @@
   <link name="base_link"></link>
   <xacro:sinsei_umiusi_control
-    high_beam_pin="$(arg high_beam_pin)"
-    low_beam_pin="$(arg low_beam_pin)"
-    ir_pin="$(arg ir_pin)"
-    indicator_led_pin="$(arg indicator_led_pin)"
+    gpiochip_device="$(arg gpiochip_device)"
+    high_beam_line_offset="$(arg high_beam_line_offset)"
+    low_beam_line_offset="$(arg low_beam_line_offset)"
+    ir_line_offset="$(arg ir_line_offset)"
+    indicator_led_line_offset="$(arg indicator_led_line_offset)"
     vesc1_id="$(arg vesc1_id)"
     vesc2_id="$(arg vesc2_id)"

File: urdf/sinsei_umiusi_control.urdf.xacro (robot description, xacro)
@@ -3,8 +3,9 @@
   <xacro:macro name="sinsei_umiusi_control"
     params="
-      high_beam_pin
-      low_beam_pin
-      ir_pin
-      indicator_led_pin
+      gpiochip_device
+      high_beam_line_offset
+      low_beam_line_offset
+      ir_line_offset
+      indicator_led_line_offset
       vesc1_id
       vesc2_id
@@ -28,9 +29,11 @@
     <xacro:imu i2c_device="${imu_i2c_device}" />
     <xacro:headlights
-      high_beam_pin="${high_beam_pin}"
-      low_beam_pin="${low_beam_pin}"
-      ir_pin="${ir_pin}" />
+      gpiochip_device="${gpiochip_device}"
+      high_beam_line_offset="${high_beam_line_offset}"
+      low_beam_line_offset="${low_beam_line_offset}"
+      ir_line_offset="${ir_line_offset}" />
     <xacro:indicator_led
-      pin="${indicator_led_pin}"
+      gpiochip_device="${gpiochip_device}"
+      line_offset="${indicator_led_line_offset}"
     />
   </xacro:macro>

File: urdf/sinsei_umiusi_control/headlights.urdf.xacro (robot description, xacro)
@@ -1,11 +1,14 @@
 <?xml version="1.0" encoding="UTF-8"?>
 <robot xmlns:xacro="http://www.ros.org/wiki/xacro" name="UMIUSI">
-  <xacro:macro name="headlights" params="high_beam_pin low_beam_pin ir_pin">
+  <xacro:macro
+    name="headlights"
+    params="gpiochip_device high_beam_line_offset low_beam_line_offset ir_line_offset">
     <ros2_control name="headlights" type="system" is_async="true">
       <hardware>
         <plugin>sinsei_umiusi_control/hardware/Headlights</plugin>
-        <param name="high_beam_pin">${high_beam_pin}</param>
-        <param name="low_beam_pin">${low_beam_pin}</param>
-        <param name="ir_pin">${ir_pin}</param>
+        <param name="gpiochip_device">${gpiochip_device}</param>
+        <param name="high_beam_line_offset">${high_beam_line_offset}</param>
+        <param name="low_beam_line_offset">${low_beam_line_offset}</param>
+        <param name="ir_line_offset">${ir_line_offset}</param>
       </hardware>
       <gpio name="headlights">

File: urdf/sinsei_umiusi_control/indicator_led.urdf.xacro (robot description, xacro)
@@ -1,9 +1,10 @@
 <?xml version="1.0" encoding="UTF-8"?>
 <robot xmlns:xacro="http://www.ros.org/wiki/xacro" name="UMIUSI">
-  <xacro:macro name="indicator_led" params="pin">
+  <xacro:macro name="indicator_led" params="gpiochip_device line_offset">
     <ros2_control name="indicator_led" type="system" is_async="true">
       <hardware>
         <plugin>sinsei_umiusi_control/hardware/IndicatorLed</plugin>
-        <param name="pin">${pin}</param>
+        <param name="gpiochip_device">${gpiochip_device}</param>
+        <param name="line_offset">${line_offset}</param>
       </hardware>
       <gpio name="indicator_led">
