Commit message: feat(bms): VESC BMSからのデータ取得に対応

File: urdf/main.urdf.xacro (robot description, xacro)
@@ -10,4 +10,5 @@
   <xacro:arg name="vesc3_id" default="'unknown'" />
   <xacro:arg name="vesc4_id" default="'unknown'" />
+  <xacro:arg name="harmony_bms_id" default="'unknown'" />
   <xacro:arg name="imu_i2c_device" default="'unknown'" />
   <xacro:include filename="sinsei_umiusi_control.urdf.xacro" />
@@ -23,4 +24,5 @@
     vesc3_id="$(arg vesc3_id)"
     vesc4_id="$(arg vesc4_id)"
+    harmony_bms_id="$(arg harmony_bms_id)"
     imu_i2c_device="$(arg imu_i2c_device)"
     mock="false"

File: urdf/sinsei_umiusi_control.urdf.xacro (robot description, xacro)
@@ -12,4 +12,5 @@
       vesc3_id
       vesc4_id
+      harmony_bms_id
       imu_i2c_device
       mock
@@ -24,4 +25,5 @@
       vesc3_id="${vesc3_id}"
       vesc4_id="${vesc4_id}"
+      harmony_bms_id="${harmony_bms_id}"
     />
     <xacro:imu i2c_device="${imu_i2c_device}" />

File: urdf/sinsei_umiusi_control/can.urdf.xacro (robot description, xacro)
@@ -2,5 +2,5 @@
 <robot xmlns:xacro="http://www.ros.org/wiki/xacro" name="UMIUSI">
   <xacro:macro name="can"
-    params="vesc1_id vesc2_id vesc3_id vesc4_id">
+    params="vesc1_id vesc2_id vesc3_id vesc4_id harmony_bms_id">
     <ros2_control name="can" type="system" is_async="true">
       <hardware>
@@ -10,4 +10,5 @@
         <param name="vesc3_id">${vesc3_id}</param>
         <param name="vesc4_id">${vesc4_id}</param>
+        <param name="harmony_bms_id">${harmony_bms_id}</param>
       </hardware>
       <xacro:macro name="thruster" params="id">
@@ -40,4 +41,7 @@
             <param name="initial_value">0.0</param>
           </state_interface>
+          <state_interface name="health" data_type="double">
+            <param name="initial_value">0.0</param>
+          </state_interface>
         </gpio>
       </xacro:macro>
@@ -46,23 +50,74 @@
       <xacro:thruster id="3" />
       <xacro:thruster id="4" />
-      <gpio name="main_power">
+      <gpio name="power_distribution">
         <command_interface name="enabled" data_type="double">
           <!-- false (Cannot use bool type due to ros2_control bug) -->
           <param name="initial_value">0.0</param>
         </command_interface>
-        <state_interface name="battery_current" data_type="double">
+      </gpio>
+      <xacro:macro name="bms_state" params="name">
+        <state_interface name="${name}" data_type="double">
           <param name="initial_value">0.0</param>
         </state_interface>
-        <state_interface name="battery_voltage" data_type="double">
-          <param name="initial_value">0.0</param>
-        </state_interface>
-        <state_interface name="temperature" data_type="double">
-          <param name="initial_value">0.0</param>
-        </state_interface>
-        <state_interface name="water_leaked" data_type="double">
-          <!-- false (Cannot use bool type due to ros2_control bug) -->
-          <param name="initial_value">0.0</param>
-        </state_interface>
-      </gpio>
+      </xacro:macro>
+      <xacro:macro name="bms_cell" params="index">
+        <xacro:bms_state name="cell_voltage_${index}" />
+        <xacro:bms_state name="cell_balancing_${index}" />
+      </xacro:macro>
+      <sensor name="bms">
+        <xacro:bms_state name="health" />
+        <xacro:bms_state name="pack_voltage" />
+        <xacro:bms_state name="charger_voltage" />
+        <xacro:bms_state name="input_current" />
+        <xacro:bms_state name="measured_current" />
+        <xacro:bms_state name="net_consumed_charge" />
+        <xacro:bms_state name="net_consumed_energy" />
+        <xacro:bms_state name="state_of_charge" />
+        <xacro:bms_state name="state_of_health" />
+        <xacro:bms_state name="cell_voltage_min" />
+        <xacro:bms_state name="cell_voltage_max" />
+        <xacro:bms_state name="cell_temperature_max" />
+        <xacro:bms_state name="charging" />
+        <xacro:bms_state name="balancing" />
+        <xacro:bms_state name="charge_allowed" />
+        <xacro:bms_state name="cell_count" />
+        <xacro:bms_cell index="0" />
+        <xacro:bms_cell index="1" />
+        <xacro:bms_cell index="2" />
+        <xacro:bms_cell index="3" />
+        <xacro:bms_cell index="4" />
+        <xacro:bms_cell index="5" />
+        <xacro:bms_cell index="6" />
+        <xacro:bms_cell index="7" />
+        <xacro:bms_cell index="8" />
+        <xacro:bms_cell index="9" />
+        <xacro:bms_cell index="10" />
+        <xacro:bms_cell index="11" />
+        <xacro:bms_state name="temperature_count" />
+        <xacro:bms_state name="temperature_0" />
+        <xacro:bms_state name="temperature_1" />
+        <xacro:bms_state name="temperature_2" />
+        <xacro:bms_state name="temperature_3" />
+        <xacro:bms_state name="temperature_4" />
+        <xacro:bms_state name="temperature_5" />
+        <xacro:bms_state name="temperature_6" />
+        <xacro:bms_state name="temperature_7" />
+        <xacro:bms_state name="temperature_8" />
+        <xacro:bms_state name="humidity_sensor_temperature" />
+        <xacro:bms_state name="relative_humidity" />
+        <xacro:bms_state name="balance_ic_temperature" />
+        <xacro:bms_state name="total_charged_charge" />
+        <xacro:bms_state name="total_charged_energy" />
+        <xacro:bms_state name="total_discharged_charge" />
+        <xacro:bms_state name="total_discharged_energy" />
+        <xacro:bms_state name="power_switch_state" />
+        <xacro:bms_state name="fault_flags" />
+        <xacro:bms_state name="data_version" />
+        <xacro:bms_state name="status_chunk_0" />
+        <xacro:bms_state name="status_chunk_1" />
+        <xacro:bms_state name="status_chunk_2" />
+        <xacro:bms_state name="status_chunk_3" />
+        <xacro:bms_state name="status_chunk_4" />
+      </sensor>
       <gpio name="led_tape">
         <command_interface name="color" data_type="double">
